Commit message: Added Files related to Env and TD3 algorithm

File: src/rl_nav_description/description/ouster_lidar.urdf.xacro (robot description, xacro)
@@ -7,5 +7,5 @@
         <parent link="${lidar_prefix}base_link"/>
         <child link="os1-32"/>
-        <origin xyz="0.0 0.0 0.3" rpy=" 0 0 0"/>
+        <origin xyz="0.0 0.0 0.45" rpy=" 0 0 0"/>
     </joint>
     <link name="os1-32">
